Commit message: Added Gripper

File: ur_description/urdf/ur10_robot.urdf (robot description, URDF)
Before this commit: robot ur10, 9 links, 8 joints
Links:
- removed link base_link
- added link arm_base_link, mass 4.0; collision mesh filename=package://ur_description/meshes/ur10/collision/base.stl; visual mesh filename=package://ur_description/meshes/ur10/visual/Base.dae
- added link robotiq_85_base_link, mass 0.636951; collision mesh filename=package://robotiq_85_description/meshes/collision/robotiq_8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; visual mesh filename=package://robotiq_85_description/meshes/visual/robotiq_85_b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
- added link robotiq_85_left_finger_link, mass 0.027309; collision mesh filename=package://robotiq_85_description/meshes/collision/robotiq_8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; visual mesh filename=package://robotiq_85_description/meshes/visual/robotiq_85_f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
- added link robotiq_85_left_finger_tip_link, mass 0.019555; collision mesh filename=package://robotiq_85_description/meshes/collision/robotiq_8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; visual mesh filename=package://robotiq_85_description/meshes/visual/robotiq_85_f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
- added link robotiq_85_left_inner_knuckle_link, mass 0.029951; collision mesh filename=package://robotiq_85_description/meshes/collision/robotiq_8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; visual mesh filename=package://robotiq_85_description/meshes/visual/robotiq_85_i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
- added link robotiq_85_left_knuckle_link, mass 0.018491; collision mesh filename=package://robotiq_85_description/meshes/collision/robotiq_8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; visual mesh filename=package://robotiq_85_description/meshes/visual/robotiq_85_k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
- added link robotiq_85_right_finger_link, mass 0.027309; collision mesh filename=package://robotiq_85_description/meshes/collision/robotiq_8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; visual mesh filename=package://robotiq_85_description/meshes/visual/robotiq_85_f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
- added link robotiq_85_right_finger_tip_link, mass 0.019555; collision mesh filename=package://robotiq_85_description/meshes/collision/robotiq_8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; visual mesh filename=package://robotiq_85_description/meshes/visual/robotiq_85_f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
- added link robotiq_85_right_inner_knuckle_link, mass 0.029951; collision mesh filename=package://robotiq_85_description/meshes/collision/robotiq_8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; visual mesh filename=package://robotiq_85_description/meshes/visual/robotiq_85_i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
- added link robotiq_85_right_knuckle_link, mass 0.018491; collision mesh filename=package://robotiq_85_description/meshes/collision/robotiq_8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; visual mesh filename=package://robotiq_85_description/meshes/visual/robotiq_85_k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
Joints:
- added joint robotiq_85_base_joint: type fixed, parent wrist_3_link, child robotiq_85_base_link, origin xyz=0.0 0.05 0.00 rpy=0 0 1.57
- added joint robotiq_85_left_finger_joint: type fixed, parent robotiq_85_left_knuckle_link, child robotiq_85_left_finger_link, origin xyz=-0.00408552455 -0.03148604435 0.0 rpy=0 0 0
- added joint robotiq_85_left_finger_tip_joint: type continuous, parent robotiq_85_left_inner_knuckle_link, child robotiq_85_left_finger_tip_link, origin xyz=0.04303959807 -0.03759940821 0.0 rpy=0.0 0.0 0.0, axis 0 0 1, limit lower=-3.14 upper=3.14 effort=0.1 velocity=100.0, mimic joint=robotiq_85_left_knuckle_joint multiplier=-1
- added joint robotiq_85_left_inner_knuckle_joint: type continuous, parent robotiq_85_base_link, child robotiq_85_left_inner_knuckle_link, origin xyz=0.06142 0.0127 0 rpy=3.14159 0.0 0.0, axis 0 0 1, limit lower=-3.14 upper=3.14 effort=0.1 velocity=100.0, mimic joint=robotiq_85_left_knuckle_joint offset=0
- added joint robotiq_85_left_knuckle_joint: type revolute, parent robotiq_85_base_link, child robotiq_85_left_knuckle_link, origin xyz=0.05490451627 0.03060114443 0.0 rpy=3.14159 0.0 0.0, axis 0 0 1, limit lower=0.0 upper=0.804 effort=1000 velocity=2.0
- added joint robotiq_85_right_finger_joint: type fixed, parent robotiq_85_right_knuckle_link, child robotiq_85_right_finger_link, origin xyz=-0.00408552455 -0.03148604435 0.0 rpy=0 0 0
- added joint robotiq_85_right_finger_tip_joint: type continuous, parent robotiq_85_right_inner_knuckle_link, child robotiq_85_right_finger_tip_link, origin xyz=0.04303959807 -0.03759940821  0.0 rpy=0.0 0.0 0.0, axis 0 0 1, limit lower=-3.14 upper=3.14 effort=0.1 velocity=100.0, mimic joint=robotiq_85_left_knuckle_joint multiplier=-1
- added joint robotiq_85_right_inner_knuckle_joint: type continuous, parent robotiq_85_base_link, child robotiq_85_right_inner_knuckle_link, origin xyz=0.06142 -0.0127 0 rpy=0 0 0, axis 0 0 1, limit lower=-3.14 upper=3.14 effort=0.1 velocity=100.0, mimic joint=robotiq_85_left_knuckle_joint offset=0
- added joint robotiq_85_right_knuckle_joint: type continuous, parent robotiq_85_base_link, child robotiq_85_right_knuckle_link, origin xyz=0.05490451627 -0.03060114443 0.0 rpy=0.0 0.0 0.0, axis 0 0 1, limit lower=-3.14 upper=3.14 effort=1000 velocity=100.0, mimic joint=robotiq_85_left_knuckle_joint
- joint ee_fixed_joint: origin xyz=0.0 0.0922 0.0 rpy=0.0 0.0 1.570796325 -> xyz=0.05 0.16 0.03 rpy=0.0 0 1.570796325
- joint shoulder_pan_joint: parent base_link -> arm_base_link
- joint world_joint: child base_link -> arm_base_link; origin xyz=0.0 0.0 0.0 rpy=0.0 0.0 0.0 -> xyz=0.0 0.0 -0.1 rpy=0.0 0.0 0.0
