Commit message: Update mobile_base_without_arm.urdf

File: ur_description/urdf/mobile_base_without_arm.urdf (robot description, URDF)
Before this commit: robot ur10, 6 links, 5 joints
Links:
- added link xtion1_frame, mass 1e-5; collision mesh filename=package://mm_description/meshes/sensors/asus_xtion_pro_live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 scale=0.001 0.001 0.001; visual mesh filename=package://mm_description/meshes/sensors/asus_xtion_pro_live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 scale=0.001 0.001 0.001
Joints:
- added joint base_link_2_xtion1_frame: type fixed, parent base_link, child xtion1_frame, origin xyz=0.32 0 0.1 rpy=0 0 0 
